Commit message: updates

File: app_simulation/o2/o2.urdf (robot description, URDF)
Before this commit: robot panda, 37 links, 36 joints
Links:
- removed link left_chassis
- removed link right_chassis
- link base_link1: geometry collision sphere radius=0.01; visual sphere radius=0.01
- link base_link2: geometry collision sphere radius=0.01; visual sphere radius=0.01
- link base_link3: geometry collision sphere radius=0.01; visual sphere radius=0.01
Joints:
- removed joint base_fixed6f
- removed joint base_fixed6f1
- removed joint left_fixed2f
- removed joint left_fixed3f
- removed joint left_fixed4f
- removed joint left_fixed5f
- removed joint left_fixed8f
- removed joint left_fixed_chassis
- removed joint right_fixed2f
- removed joint right_fixed3f
- removed joint right_fixed4f
- removed joint right_fixed5f
- removed joint right_fixed8
- removed joint right_fixed8f
- removed joint right_fixed_chassis
- added joint base_fixed_6f: type fixed, parent base_link6, child base_link6f, origin xyz=0 0 0 rpy=0 0 0, axis 0 0 1, limit lower=-2.8973 upper=2.8973 effort=87 velocity=2.1750
- added joint base_fixed_6f1: type fixed, parent base_link6f, child base_link6f1, origin xyz=0 0 0 rpy=0 0 0, axis 0 0 1, limit lower=-2.8973 upper=2.8973 effort=87 velocity=2.1750
- added joint left_fixed_2f: type fixed, parent left_link2, child left_link2f, origin xyz=0 0 0 rpy=0 0 0, axis 0 0 1, limit lower=-2.8973 upper=2.8973 effort=87 velocity=2.1750
- added joint left_fixed_3f: type fixed, parent left_link3, child left_link3f, origin xyz=0 0 0 rpy=0 0 0, axis 0 0 1, limit lower=-2.8973 upper=2.8973 effort=87 velocity=2.1750
- added joint left_fixed_4f: type fixed, parent left_link4, child left_link4f, origin xyz=0 0 0 rpy=0 0 0, axis 0 0 1, limit lower=-2.8973 upper=2.8973 effort=87 velocity=2.1750
- added joint left_fixed_5f: type fixed, parent left_link5, child left_link5f, origin xyz=0 0 0 rpy=0 0 0, axis 0 0 1, limit lower=-2.8973 upper=2.8973 effort=87 velocity=2.1750
- added joint left_fixed_8f: type fixed, parent left_link8, child left_link8f, origin xyz=0 0 0 rpy=0 0 0, axis 0 0 1, limit lower=-2.8973 upper=2.8973 effort=87 velocity=2.1750
- added joint right_fixed_2f: type fixed, parent right_link2, child right_link2f, origin xyz=0 0 0 rpy=0 0 0, axis 0 0 1, limit lower=-2.8973 upper=2.8973 effort=87 velocity=2.1750
- added joint right_fixed_3f: type fixed, parent right_link3, child right_link3f, origin xyz=0 0 0 rpy=0 0 0, axis 0 0 1, limit lower=-2.8973 upper=2.8973 effort=87 velocity=2.1750
- added joint right_fixed_4f: type fixed, parent right_link4, child right_link4f, origin xyz=0 0 0 rpy=0 0 0, axis 0 0 1, limit lower=-2.8973 upper=2.8973 effort=87 velocity=2.1750
- added joint right_fixed_5f: type fixed, parent right_link5, child right_link5f, origin xyz=0 0 0 rpy=0 0 0, axis 0 0 1, limit lower=-2.8973 upper=2.8973 effort=87 velocity=2.1750
- added joint right_fixed_8: type fixed, parent right_link7, child right_link8, origin xyz=0 -0.23675 0 rpy=1.5707963 0 0, axis 0 0 1, limit lower=-2.8973 upper=2.8973 effort=87 velocity=2.1750
- added joint right_fixed_8f: type fixed, parent right_link8, child right_link8f, origin xyz=0 0 0 rpy=0 0 0, axis 0 0 1, limit lower=-2.8973 upper=2.8973 effort=87 velocity=2.1750
- joint left_joint1: origin xyz=0 0 0 rpy=0 1.5707963 -1.5707963 -> xyz=0.58 0.2 0 rpy=0 1.5707963 -2.536194; parent left_chassis -> base_link6
- joint right_joint1: origin xyz=0 0 0 rpy=0 1.5707963 -1.5707963 -> xyz=0.58 -0.2 0 rpy=1.5707963 1.5707963 0.785398; parent right_chassis -> base_link6
